File: MagicStick_hw/MagicStick.sch (KiCad schematic (older format))
At the start: 57 parts, among them SW3 BUTTON

Commit message: + Stick PCB layout done
Parts:
- removed DD?: STM32L431CxTx, LQFP_TQFP:LQFP48, symbol st_kl:STM32L431CxTx
- removed Q?: BC848, symbol Transistors_kl:NPN
- removed R5: 100R, Resistors:RES_0603, symbol Tittar_kl:R
- removed RP1, RP2, RP3, RP4: REFPOINT, PCB:REF_POINT_1MM, symbol pcb_details:REFPOINT
- removed TP2: TESTPOINT, PCB:TESTPOINT_1MM, symbol pcb_details:TESTPOINT
- removed XL6: CONN_4, Connectors:PLS-4-Long, symbol Connectors_kl:CONN_4
- added C1, C2: 10n, Capacitors:CAP_0603, symbol Tittar_kl:C
- added C15, C23, C24, C25, C3, C30, C31: 10u, Capacitors:CAP_0603, symbol Tittar_kl:C
- added C18, C32, C33, C7: 1u, Capacitors:CAP_0603, symbol Tittar_kl:C
- added C26: 0.1u, Capacitors:CAP_0603, symbol Tittar_kl:C
- added C37, C38: *, Capacitors:CAP_0402, symbol Tittar_kl:C
- added D1, D3: NSR0320, Diodes:SOD323, symbol Tittar_kl:D_Shottky
- added D2: LED, LEDs:Cree_J3030, symbol Tittar_kl:LED
- added D4: LED, LEDs:LED_0603, symbol Tittar_kl:LED
- added DA1: ST1CC40_SO8, SO_DIL_TSSOP:SO8_150MIL, symbol Power_kl:ST1CC40_SO8
- added DA2: TP4056, SO_DIL_TSSOP:SO8_150MIL, symbol Power_kl:TP4056
- added DA3: MCP1700, SOT:SOT23-3A, symbol Power_kl:MCP1700
- added DD1: STM32L433Cx, LQFP_TQFP:LQFP48, symbol st_kl:STM32L433Cx
- added L4: 2.2uH, Inductors:IND_SRN2512, symbol Tittar_kl:L
- added L5: *, Inductors:IND_0402, symbol Tittar_kl:L
- added M1: MOTOR_NO_CONTACTS, Installation:Motor_no_Contacts, symbol pcb_details:MOTOR_NO_CONTACTS
- added Q1, Q10, Q11, Q12, Q3, Q4, Q5, Q8, Q9: MMBT2222, SOT:SOT23-3, symbol Transistors_kl:NPN
- added Q2: IRLML6401, SOT:SOT23-3, symbol Transistors_kl:P_3PIN
- added Q6, Q7: LED_RGB_6PIN_PAD, LEDs:EpistarRGB, symbol Tittar_kl:LED_RGB_6PIN_PAD
- added R1: 1M, Resistors:RES_0603, symbol Tittar_kl:R
- added R12: 4k7, Resistors:RES_0603, symbol Tittar_kl:R
- added R13, R27: 1k, Resistors:RES_0603, symbol Tittar_kl:R
- added R15, R16, R2, R23, R24, R28, R29: 510R, Resistors:RES_0603, symbol Tittar_kl:R
- added R19, R20, R25, R26, R30, R31: 1R0, Resistors:RES_0805, symbol Tittar_kl:R
- added R6: 10k, Resistors:RES_0603, symbol Tittar_kl:R
- added R7: 100k, Resistors:RES_0603, symbol Tittar_kl:R
- added R8: 0R2, Resistors:RES_1206, symbol Tittar_kl:R
- added R9: 0R1, Resistors:RES_1206, symbol Tittar_kl:R
- added TP1: TESTPOINT, PCB:TESTPOINT_1MM, symbol pcb_details:TESTPOINT
- added XL4: USB_MICRO, Connectors:USBmicro_MOLEX_1050170001, symbol Connectors_kl:USB_MINI_B
- added XL5: CONN_2, Connectors:PBS-2, symbol Connectors_kl:CONN_2
- added XL7, XL8: CONN_1, PCB:Oval3x1.5, symbol Connectors_kl:CONN_1
- BLN1: symbol RF_ICs:BALUN868JOHANSON -> RFICs:BALUN868JOHANSON
- DD4: renamed from DD3; symbol RF_ICs:CC1101 -> RFICs:CC1101
- Logo1: footprint Pictures:Ostranna_12d7_10d1 -> Pictures:Ostranna_8x8
- R3: value 100R -> 100k
- R4: value 100R -> 1R0; footprint Resistors:RES_0603 -> Resistors:RES_0805
- XL2: footprint Connectors:PLS-1Square -> PCB:Oval3x1.5
- XL3: footprint Connectors:SIL1_ROUND_1MM8 -> PCB:Oval3x1.5
- gave numbers to parts that had none: 13
- renumbered C7 to C10, C8 to C11, C9 to C12, C10 to C13, C11 to C14, C12 to C16, C13 to C17, C14 to C19, C15 to C20, C16 to C21, C20 to C27, C21 to C29, C17 to C34, C18 to C35, C19 to C36, C3 to C4, C5 to C8, C6 to C9, L2 to L1, L3 to L2, R2 to R14, R8 to R17, SW3 to SW1, TP1 to TP2, XTAL1 to XTAL2
Connections:
- net labels added: 5V_MID, 5V_USB, IR_CARRIER, IR_LEVEL, IS_CHARGING, LUMOS_CTRL, PwrUnst, SW1, USB_DM, USB_DP, VIBRO_CTRL, VIBRO_OUT, WHITE_A, WHITE_C
- net labels removed: ANT1, CC_GDO2, IR_CTRL
- wire segments 235 -> 424
- no-connect marks 9 -> 7
Other:
- note added: "Battery connector"
- note added: "Battery or USB"
- note added: "Charger\n4k7 => 270 mA"
- note added: "DAC1"
- note added: "Debug \noutput"
- note added: "I2C1"
- note added: "IR TX"
- note added: "LPTIM1 OUT OpenDrain"
- note added: "Lumos"
- note added: "MCU power"
- note added: "Periphery\n\nDAC1: IR power\nPA0: WKUP1 by BTN\nPC13: WKUP2 by ACG\nPA2: WKUP4 by Charging\nLPTIM1: IR carrier (56kHz)\nT1 C1,2,3: RGB LED\nT2 (32bit): systick\nT15 C2: Vibro\nT16 C1: Lumos\nI2C1: EEPROM\nSPI1: CC1101\nSPI2: ACG\nUSART1: Debug UART\n\nDMA1\nC1: ADC\nC4: SPI2_RX\nC5: SPI2_TX\nC6: I2C1_TX\nC7: I2C1_RX\n\nDMA2:\nC4: DAC\nC5: TIM7 (for IR)\nC6: USART1_TX\nC7: USART1_RX"
- note added: "Power"
- note added: "Pull-up when reset"
- note added: "RGB LED"
- note added: "SPI2"
- note added: "T15C2"
- note added: "T16C1"
- note added: "T1C1"
- note added: "T1C2"
- note added: "T1C3"
- note added: "USART1"
- note added: "Vibro"
- note added: "WKUP1"
- note added: "WKUP2"
- note added: "WKUP4"
- note removed: "Periphery\n\nPA0: WKUP\nT3 C2, 3, 4: LED RGB\nSPI1: CC\nSPI2: ACG\nUART2: Debug UART\n\nDMA\nC1: ADC\nC4: SPI2_RX\nC5: SPI2_TX\nC6: USART2_RX\nC7: USART2_TX"
- note removed: "RGB LED connector"
- moved on the sheet: ANT1, BLN1, C10, C11, C12, C13, C14, C16, C17, C19, C20, C21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

Commit message: Ready for factory
Parts:
- ANT1: footprint Antennas:ANT_868_10d4x36 -> Antennas:MagicStick
Changed lines of the file:
@@
 F 0 "ANT1" H 18593 2137 60  0000 C CNN
 F 1 "ANT_PCB_MONO" H 18593 2031 60  0000 C CNN
-F 2 "Antennas:ANT_868_10d4x36" H 18200 2000 60  0001 C CNN
+F 2 "Antennas:MagicStick" H 18200 2000 60  0001 C CNN
 F 3 "" H 18300 2100 60  0001 C CNN
 F 4 "0" H 18400 2200 60  0001 C CNN "Price"

Commit message: .
Connections:
- net +BATT: now also D3.C
- net VIBRO_OUT: now also D3.A
- net +3.3V renamed +3v3
Changed lines of the file:
@@
 	0    1    -1   0
-$EndComp
-$Comp
-L power:+3.3V #PWR015
-U 1 1 5C471384
-P 3150 5800
-F 0 "#PWR015" H 3150 5760 30  0001 C CNN
-F 1 "+3.3V" H 3187 5868 30  0000 C CNN
-F 2 "" H 3150 5800 60  0000 C CNN
-F 3 "" H 3150 5800 60  0000 C CNN
-	1    3150 5800
-	-1   0    0    -1
-$EndComp
-$Comp
-L power:+3.3V #PWR014
-U 1 1 5C471853
-P 3100 7800
-F 0 "#PWR014" H 3100 7760 30  0001 C CNN
-F 1 "+3.3V" H 3137 7868 30  0000 C CNN
-F 2 "" H 3100 7800 60  0000 C CNN
-F 3 "" H 3100 7800 60  0000 C CNN
-	1    3100 7800
-	-1   0    0    -1
 $EndComp
 Wire Wire Line
@@
 Wire Wire Line
 	1700 6350 1850 6350
-$Comp
-L power:+3.3V #PWR072
-U 1 1 5C300BF4
-P 12550 14850
-F 0 "#PWR072" H 12550 14810 30  0001 C CNN
-F 1 "+3.3V" H 12630 14880 30  0000 C CNN
-F 2 "" H 12550 14850 60  0001 C CNN
-F 3 "" H 12550 14850 60  0001 C CNN
-	1    12550 14850
-	1    0    0    -1
-$EndComp
 $Comp
 L Power_kl:TP4056 DA2
@@
 Text Notes 11350 5300 0    79   ~ 0
 Vibro
-Wire Wire Line
-	11800 5750 11800 5650
 Connection ~ 11800 5650
-Wire Wire Line
-	11800 6150 11800 6250
 Connection ~ 11800 6250
 $Comp
@@
 Wire Wire Line
 	2850 10450 2850 10850
+Wire Wire Line
+	11800 5650 11800 5800
+Wire Wire Line
+	11800 6100 11800 6250
+$Comp
+L power:+3v3 #PWR?
+U 1 1 5C831376
+P 3150 5800
+F 0 "#PWR?" H 3150 5760 30  0001 C CNN
+F 1 "+3v3" H 3187 5868 30  0000 C CNN
+F 2 "" H 3150 5800 60  0000 C CNN
+F 3 "" H 3150 5800 60  0000 C CNN
+	1    3150 5800
+	-1   0    0    -1
+$EndComp
+$Comp
+L power:+3v3 #PWR?
+U 1 1 5C831DC4
+P 3100 7800
+F 0 "#PWR?" H 3100 7760 30  0001 C CNN
+F 1 "+3v3" H 3137 7868 30  0000 C CNN
+F 2 "" H 3100 7800 60  0000 C CNN
+F 3 "" H 3100 7800 60  0000 C CNN
+	1    3100 7800
+	-1   0    0    -1
+$EndComp
+$Comp
+L power:+3v3 #PWR?
+U 1 1 5C89240B
+P 12550 14850
+F 0 "#PWR?" H 12550 14810 30  0001 C CNN
+F 1 "+3v3" H 12587 14918 30  0000 C CNN
+F 2 "" H 12550 14850 60  0000 C CNN
+F 3 "" H 12550 14850 60  0000 C CNN
+	1    12550 14850
+	1    0    0    -1
+$EndComp
 Wire Bus Line
 	14200 1350 14200 2450
