File: MagicStick_hw/MagicStick.kicad_pcb (KiCad board)
At the start: 2 copper layers, 259.1 x 13.5 mm, 113 parts, among them M1 MOTOR_NO_CONTACTS, Q1 MMBT2222, Q10 MMBT2222, Q11 MMBT2222, Q12 MMBT2222, Q2 IRLML6401, Q3 MMBT2222, Q4 MMBT2222, Q5 MMBT2222, Q6 LED_RGB_6PIN_PAD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

Commit message: Minor
Parts:
- moved C38 3.70 mm to (180.6, 104.2), turned to 270 degrees
- moved Q1 1.70 mm to (68.8, 100.0)
- moved R2 1.70 mm to (72.1, 101.7)
- moved R3 1.70 mm to (72.1, 100.0)
- moved R4 1.70 mm to (72.5, 98.1)
- moved C15 0.60 mm to (65.3, 97.6)
- moved C3 0.60 mm to (65.3, 99.2)
- moved C31 0.60 mm to (65.3, 100.8)
- moved R7 0.60 mm to (65.3, 102.4)
- moved C18 0.60 mm to (52.9, 102.3)
- moved C24 0.60 mm to (50.3, 98.5)
- moved C25 0.60 mm to (50.3, 101.5)
- moved DA1 0.60 mm to (58.9, 100.0)
- moved L4 0.60 mm to (52.9, 100.0)
- moved C26 0.60 mm to (48.7, 98.5)
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Changed lines of the file:
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@@
   (general
     (thickness 1.6)
-    (drawings 17)
+    (drawings 23)
     (tracks 0)
     (zones 0)
@@
     (solder_mask_min_width 0.18)
     (aux_axis_origin 0 0)
-    (visible_elements 7FFFFE1F)
+    (visible_elements 7FFFF61F)
     (pcbplotparams
       (layerselection 0x010f0_ffffffff)
@@
   )
   (module Capacitors:CAP_0603 (layer F.Cu)
-    (at 65.9 99.2 180)
+    (at 65.3 99.2 180)
     (attr smd)
     (fp_text reference C3 (at 0 0 180) (layer F.SilkS)
@@
   )
   (module Capacitors:CAP_0603 (layer F.Cu)
-    (at 183 103.6 180)
+    (at 183 104 180)
     (attr smd)
     (fp_text reference C11 (at 0 0 180) (layer F.SilkS)
@@
   )
   (module Capacitors:CAP_0603 (layer F.Cu)
-    (at 65.9 97.6)
+    (at 65.3 97.6)
     (attr smd)
     (fp_text reference C15 (at 0 0) (layer F.SilkS)
@@
   )
   (module Capacitors:CAP_0603 (layer F.Cu)
-    (at 53.5 102.3 180)
+    (at 52.9 102.3 180)
     (attr smd)
     (fp_text reference C18 (at 0 0 180) (layer F.SilkS)
@@
   )
   (module Capacitors:CAP_0603 (layer F.Cu)
-    (at 50.9 98.5 90)
+    (at 50.3 98.5 90)
     (attr smd)
     (fp_text reference C24 (at 0 0 90) (layer F.SilkS)
@@
   )
   (module Capacitors:CAP_0603 (layer F.Cu)
-    (at 50.9 101.5 270)
+    (at 50.3 101.5 270)
     (attr smd)
     (fp_text reference C25 (at 0 0 270) (layer F.SilkS)
@@
   )
   (module Capacitors:CAP_0603 (layer F.Cu)
-    (at 49.3 98.5 90)
+    (at 48.7 98.5 90)
     (attr smd)
     (fp_text reference C26 (at 0 0 90) (layer F.SilkS)
@@
   )
   (module Capacitors:CAP_0603 (layer F.Cu)
-    (at 65.9 100.8 180)
+    (at 65.3 100.8 180)
     (attr smd)
     (fp_text reference C31 (at 0 0 180) (layer F.SilkS)
@@
   )
   (module Capacitors:CAP_0402 (layer F.Cu)
-    (at 181.7 100.5 90)
+    (at 181.7 101 90)
     (attr smd)
     (fp_text reference C37 (at 0 0 90) (layer F.SilkS)
@@
   )
   (module Capacitors:CAP_0402 (layer F.Cu)
-    (at 180.5 100.5 90)
+    (at 180.6 104.2 270)
     (attr smd)
-    (fp_text reference C38 (at 0 0 90) (layer F.SilkS)
+    (fp_text reference C38 (at 0 0 270) (layer F.SilkS)
       (effects (font (size 0.5 0.5) (thickness 0.1)))
     )
-    (fp_text value * (at 0 1.15 90) (layer F.Fab)
+    (fp_text value * (at 0 1.15 270) (layer F.Fab)
       (effects (font (size 0.6 0.6) (thickness 0.15)))
     )
@@
     (fp_line (start 0.95 0.45) (end -0.95 0.45) (layer F.SilkS) (width 0.15))
     (fp_line (start -0.95 0.45) (end -0.95 -0.45) (layer F.SilkS) (width 0.15))
-    (pad 1 smd rect (at -0.5 0 90) (size 0.6 0.7) (layers F.Cu F.Paste F.Mask)
+    (pad 1 smd rect (at -0.5 0 270) (size 0.6 0.7) (layers F.Cu F.Paste F.Mask)
       (net 27 "Net-(ANT1-Pad1)"))
-    (pad 2 smd rect (at 0.5 0 90) (size 0.6 0.7) (layers F.Cu F.Paste F.Mask)
+    (pad 2 smd rect (at 0.5 0 270) (size 0.6 0.7) (layers F.Cu F.Paste F.Mask)
       (net 1 GND))
     (model ${KICAD_SYMBOL_DIR}/3d/Capacitors/C_0402.step
@@
   )
   (module SO_DIL_TSSOP:SO8_150MIL (layer F.Cu)
-    (at 59.5 100 270)
+    (at 58.9 100 270)
     (descr "SO8 150mil")
     (attr smd)
@@
   )
   (module Inductors:IND_SRN2512 (layer F.Cu)
-    (at 53.5 100)
+    (at 52.9 100)
     (attr smd)
     (fp_text reference L4 (at 0.05 -1.75) (layer F.SilkS)
@@
   )
   (module Inductors:IND_0402 (layer F.Cu)
-    (at 181.2 102.1 180)
+    (at 181.2 102.6 180)
     (attr smd)
     (fp_text reference L5 (at 0 -1.1 180) (layer F.SilkS)
@@
   )
   (module SOT:SOT23-3 (layer F.Cu)
-    (at 70.5 100 270)
+    (at 68.8 100 270)
     (descr "Module SOT23")
     (attr smd)
@@
   )
   (module Resistors:RES_0603 (layer F.Cu)
-    (at 73.8 101.7 180)
+    (at 72.1 101.7 180)
     (attr smd)
     (fp_text reference R2 (at 0 0 180) (layer F.SilkS)
@@
   )
   (module Resistors:RES_0603 (layer F.Cu)
-    (at 73.8 100)
+    (at 72.1 100)
     (attr smd)
     (fp_text reference R3 (at 0 0) (layer F.SilkS)
@@
   )
   (module Resistors:RES_0805 (layer F.Cu)
-    (at 74.2 98.1)
+    (at 72.5 98.1)
     (attr smd)
     (fp_text reference R4 (at 0.2 0.1) (layer F.SilkS)
@@
   )
   (module Resistors:RES_0603 (layer F.Cu)
-    (at 65.9 102.4)
+    (at 65.3 102.4)
     (attr smd)
     (fp_text reference R7 (at 0 0) (layer F.SilkS)
@@
     )
   )
+  (dimension 1.5 (width 0.15) (layer Dwgs.User)
+    (gr_text "1.500 mm" (at 265.9 106 270) (layer Dwgs.User)
+      (effects (font (size 1 1) (thickness 0.15)))
+    )
+    (feature1 (pts (xy 269.5 106.75) (xy 266.613579 106.75)))
+    (feature2 (pts (xy 269.5 105.25) (xy 266.613579 105.25)))
+    (crossbar (pts (xy 267.2 105.25) (xy 267.2 106.75)))
+    (arrow1a (pts (xy 267.2 106.75) (xy 266.613579 105.623496)))
+    (arrow1b (pts (xy 267.2 106.75) (xy 267.786421 105.623496)))
+    (arrow2a (pts (xy 267.2 105.25) (xy 266.613579 106.376504)))
+    (arrow2b (pts (xy 267.2 105.25) (xy 267.786421 106.376504)))
+  )
+  (dimension 46 (width 0.15) (layer Dwgs.User)
+    (gr_text "46.000 mm" (at 246.5 109.15) (layer Dwgs.User)
+      (effects (font (size 1 1) (thickness 0.15)))
+    )
+    (feature1 (pts (xy 223.5 105.25) (xy 223.5 108.436421)))
+    (feature2 (pts (xy 269.5 105.25) (xy 269.5 108.436421)))
+    (crossbar (pts (xy 269.5 107.85) (xy 223.5 107.85)))
+    (arrow1a (pts (xy 223.5 107.85) (xy 224.626504 107.263579)))
+    (arrow1b (pts (xy 223.5 107.85) (xy 224.626504 108.436421)))
+    (arrow2a (pts (xy 269.5 107.85) (xy 268.373496 107.263579)))
+    (arrow2b (pts (xy 269.5 107.85) (xy 268.373496 108.436421)))
+  )
+  (dimension 9.6 (width 0.15) (layer Dwgs.User)
+    (gr_text "9.600 mm" (at 274.3 109.149999) (layer Dwgs.User)
+      (effects (font (size 1 1) (thickness 0.15)))
+    )
+    (feature1 (pts (xy 279.1 105.25) (xy 279.1 108.43642)))
+    (feature2 (pts (xy 269.5 105.25) (xy 269.5 108.43642)))
+    (crossbar (pts (xy 269.5 107.849999) (xy 279.1 107.849999)))
+    (arrow1a (pts (xy 279.1 107.849999) (xy 277.973496 108.43642)))
+    (arrow1b (pts (xy 279.1 107.849999) (xy 277.973496 107.263578)))
+    (arrow2a (pts (xy 269.5 107.849999) (xy 270.626504 108.43642)))
+    (arrow2b (pts (xy 269.5 107.849999) (xy 270.626504 107.263578)))
+  )
+  (dimension 13.5 (width 0.15) (layer Dwgs.User)
+    (gr_text "13.500 mm" (at 283.1 100 270) (layer Dwgs.User)
+      (effects (font (size 1 1) (thickness 0.15)))
+    )
+    (feature1 (pts (xy 279.1 106.75) (xy 282.386421 106.75)))
+    (feature2 (pts (xy 279.1 93.25) (xy 282.386421 93.25)))
+    (crossbar (pts (xy 281.8 93.25) (xy 281.8 106.75)))
+    (arrow1a (pts (xy 281.8 106.75) (xy 281.213579 105.623496)))
+    (arrow1b (pts (xy 281.8 106.75) (xy 282.386421 105.623496)))
+    (arrow2a (pts (xy 281.8 93.25) (xy 281.213579 94.376504)))
+    (arrow2b (pts (xy 281.8 93.25) (xy 282.386421 94.376504)))
+  )
+  (dimension 160 (width 0.15) (layer Dwgs.User)
+    (gr_text "160.000 mm" (at 100 112) (layer Dwgs.User)
+      (effects (font (size 1 1) (thickness 0.15)))
+    )
+    (feature1 (pts (xy 20 103.5) (xy 20 111.286421)))
+    (feature2 (pts (xy 180 103.5) (xy 180 111.286421)))
+    (crossbar (pts (xy 180 110.7) (xy 20 110.7)))
+    (arrow1a (pts (xy 20 110.7) (xy 21.126504 110.113579)))
+    (arrow1b (pts (xy 20 110.7) (xy 21.126504 111.286421)))
+    (arrow2a (pts (xy 180 110.7) (xy 178.873496 110.113579)))
+    (arrow2b (pts (xy 180 110.7) (xy 178.873496 111.286421)))
+  )
+  (dimension 99.1 (width 0.15) (layer Dwgs.User)
+    (gr_text "99.100 mm" (at 229.55 111.999999) (layer Dwgs.User)
+      (effects (font (size 1 1) (thickness 0.15)))
+    )
+    (feature1 (pts (xy 279.1 104.5) (xy 279.1 111.28642)))
+    (feature2 (pts (xy 180 104.5) (xy 180 111.28642)))
+    (crossbar (pts (xy 180 110.699999) (xy 279.1 110.699999)))
+    (arrow1a (pts (xy 279.1 110.699999) (xy 277.973496 111.28642)))
+    (arrow1b (pts (xy 279.1 110.699999) (xy 277.973496 110.113578)))
+    (arrow2a (pts (xy 180 110.699999) (xy 181.126504 111.28642)))
+    (arrow2b (pts (xy 180 110.699999) (xy 181.126504 110.113578)))
+  )
   (gr_line (start 180 95.5) (end 180 104.5) (layer Dwgs.User) (width 0.15))

Commit message: Ready for factory
Parts:
- ANT1: footprint Antennas:ANT_868_10d4x36 -> Antennas:MagicStick
- C1: moved to F.Cu
- C30: moved to B.Cu
- moved ANT1 26.6 mm to (180.0, 100.0)
- moved R27 11.1 mm to (276.7, 105.5)
- moved D4 11.0 mm to (276.8, 105.5)
- moved C30 10.7 mm to (270.6, 95.9), turned to 90 degrees
- moved C33 9.66 mm to (216.0, 104.7)
- moved D1 9.60 mm to (273.5, 104.0), turned to 90 degrees
- moved C32 9.35 mm to (221.7, 104.4), turned to 90 degrees
- moved DA3 9.07 mm to (218.9, 104.4)
- moved R6 8.71 mm to (271.0, 104.8), turned to 270 degrees
- moved R8 8.57 mm to (273.4, 95.0), turned to 0 degrees
- moved R12 7.80 mm to (273.3, 105.5)
- moved C2 7.62 mm to (273.5, 97.7)
- moved Q2 7.58 mm to (271.3, 104.3), turned to 90 degrees
- moved C28 6.99 mm to (219.8, 98.2)
- moved R1 6.98 mm to (277.6, 99.2), turned to 270 degrees
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Routing:
- net GND: track 0.00 -> 534.6 mm, vias 0 -> 61
- net +BATT: track 0.00 -> 314.5 mm, vias 0 -> 8
- net /BLUE_LED: track 0.00 -> 172.8 mm, vias 0 -> 3
- net /RED_LED: track 0.00 -> 171.4 mm, vias 0 -> 3
- net /GREEN_LED: track 0.00 -> 169.1 mm, vias 0 -> 3
- net /LUMOS_CTRL: track 0.00 -> 160.8 mm, vias 0 -> 4
- net /IR_CARRIER: track 0.00 -> 158.6 mm
- net /IR_LEVEL: track 0.00 -> 145.4 mm, vias 0 -> 2
- net /IS_CHARGING: track 0.00 -> 89.8 mm, vias 0 -> 1
- net PwrMCU: track 0.00 -> 69.7 mm, vias 0 -> 6
- net /USB_DM: track 0.00 -> 68.7 mm
- net /USB_DP: track 0.00 -> 68.6 mm
- net PwrUnst: track 0.00 -> 55.1 mm
- net VCC: track 0.00 -> 54.7 mm, vias 0 -> 7
- net Net-(Q1-Pad3): track 0.00 -> 46.8 mm, vias 0 -> 1
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- added copper zone on B.Cu, net +BATT
- added copper zone on In1.Cu, net +BATT
- added copper zone on In2.Cu, net +BATT
- added copper zone on B.Cu, net GND
- added copper zone on F.Cu, net GND
- added copper zone on In1.Cu, net GND
- added copper zone on In2.Cu, net GND
- added copper zone on F.Cu, net PwrUnst
Other:
- copper layers 2 -> 4
- net class Wide: clearance 0.2 -> 0.18
- rule pad_to_mask_clearance: 0.1 -> 0.06
- rule solder_mask_min_width: 0.18 -> 0.15
- rule via_min_size: 0.4 -> 0.7
- board text added: "+"
- board text added: "-"
